File: hardware/gdoor-din/esp32.kicad_pcb (KiCad board)
At the start: 4 copper layers, 50 x 85 mm, 198 parts, among them J1 PlugIn_Terminal_Screw, J101 USB-C, J102 HR911105A, J103 EXP, J4 5V_IN, Q1 MMBT5401, Q2 MMBT2222A, SW101 RESET, SW102 BOOT, U1 TLV9351, U101 ESP32-S3-WROOM-1-N8R2, U102 USBLC6-2SC6, U103 AMS1117-3.3, U104 W5500, U2 LMV321, U3 LMV321, U5 ES8374, U6 LM393, U7 AMS1117-3.3, Y101 25MHz

Commit message: gdoor-din: give SW101/SW102 one value so JLC merges their BOM line
Both buttons are the same part (C318884); the values RESET and BOOT
made two BOM lines matched to one part, which JLC flags. Both are now
"TL3342"; the schematic net labels still say which is which.

Co-Authored-By: Claude Opus 5.5 <noreply@anthropic.com>
Parts:
- SW101: value RESET -> TL3342
- SW102: value BOOT -> TL3342
Changed lines of the file:
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@@
 			)
 		)
-		(property "Value" "RESET"
+		(property "Value" "TL3342"
 			(at 0 3.75 90)
 			(layer "F.Fab")
@@
 			)
 		)
-		(property "Value" "BOOT"
+		(property "Value" "TL3342"
 			(at 0 3.75 90)
 			(layer "F.Fab")

Commit message: gdoor-din: route Ethernet RX and USB D+/D- as coupled, length-matched pairs
Both pairs were routed as two independent nets (USB 3.3 mm and the
Ethernet receive chain ~2-4 mm apart, with the RX legs on different
layers and up to 11 vias). Now:

- RX passives re-placed as a mirrored cluster so no leg has to cross
  the other on one layer: R117/R118 stand side by side with their chip
  pads at the top; C121<->C122 and R119<->R120 swapped so P and N each
  stay on their own side. C124 (shield cap) moved out of the way.
- Pairs routed coupled at 0.2 mm / 0.15 mm gap (~100 ohm differential
  over the In1 GND plane): RX chip side on F.Cu, RX jack side and both
  USB segments on B.Cu, with 45-degree splays where they fan out to pads.
- Skew tuned with 45-degree bumps on the shorter leg. Pad-to-pad:
  USB J101 -> module 61.25 / 61.02 mm (0.23 mm), Ethernet RX chip ->
  RJ45 42.26 / 43.25 mm (1.0 mm, ~6 ps; no room left for more bumps).
- Displaced nets re-routed, GND pours and stitching re-made, silk
  re-placed (C123's reference now hidden as well).

kicad-cli DRC: 0 errors, 0 unconnected, parity clean, silk clean.

Co-Authored-By: Claude Opus 5.5 <noreply@anthropic.com>
Parts:
- moved R118 24.9 mm to (120.5, 101.2), turned to -90 degrees
- moved C124 5.95 mm to (116.1, 104.8)
- moved C121 2.97 mm to (116.8, 100.0)
- moved C122 2.97 mm to (117.4, 103.0)
- moved R120 1.89 mm to (114.5, 102.0), turned to 90 degrees
- moved R119 1.89 mm to (114.5, 100.1), turned to 0 degrees
- moved R117 1.78 mm to (119.3, 101.2), turned to -90 degrees
Routing:
- net /MCU, USB, Power, Ethernet/ETH_RXP_C: track 34.4 -> 6.67 mm, vias 5 -> 2
- net /MCU, USB, Power, Ethernet/ETH_RXP_CHIP: track 40.2 -> 19.7 mm, vias 5 -> 0
- net /MCU, USB, Power, Ethernet/USB_DN: track 47.6 -> 66.5 mm, vias 5 -> 6
- net /MCU, USB, Power, Ethernet/USB_DP: track 44.4 -> 62.3 mm, vias 4 -> 5
- net /MCU, USB, Power, Ethernet/ETH_SHIELD: track 33.1 -> 23.3 mm
- net +5V: track 129.6 -> 123.2 mm
- net /MCU, USB, Power, Ethernet/ETH_RD_P: track 13.1 -> 19.3 mm
- net /MCU, USB, Power, Ethernet/ETH_RD_N: track 15.1 -> 19.6 mm, vias 0 -> 2
- net /MCU, USB, Power, Ethernet/ETH_RXN_C: track 8.53 -> 5.98 mm
- net /MCU, USB, Power, Ethernet/ETH_EXRES: track 19.6 -> 21.6 mm
- net /MCU, USB, Power, Ethernet/ETH_ACTLED: track 14.1 -> 15.7 mm, vias 2 -> 4
- net /MCU, USB, Power, Ethernet/ETH_RXN_CHIP: track 18.9 -> 19.4 mm, vias 2 -> 0
- net /MCU, USB, Power, Ethernet/+3.3V_ETHA: track 70.7 -> 70.6 mm, vias 4 -> 6
- net GND: vias 281 -> 280
