File: hardware/gdoor-din/esp32.kicad_sch (KiCad schematic)
At the start: 149 parts, among them J1 PlugIn_Terminal_Screw, J4 PlugIn_Terminal_01x02, Q4 MMBT5401, Q5 MMBT2222A, U4 TLV9351, U5 ES8374, U5 LMV321, U6 LM393, U6 LMV321, U7 AMS1117-3.3

Commit message: DIN board: clean up main sheet, fit 5 V input terminal
After re-saving in KiCad (which refreshed 52 stale cached references from an
older copied-in project), remove the leftover ESP32-S3 devkit symbol, its
orphaned power symbols, dangling wire stubs and bus entries, and convert the
bus/audio signal labels to global labels so they connect to the MCU sheet.
J4 (5 V screw terminal via D2) now uses the 3.5 mm terminal C695629 like J1.

ERC: 0 errors on both sheets; remaining warnings are the original drawing's
off-grid endpoints and the unused RX_DAC label (R56 not fitted).
Still to do in KiCad: untick DNP / tick 'in BOM' on J4.

Co-Authored-By: Claude Opus 5.5 <noreply@anthropic.com>
Parts:
- removed U4: (no value), Library:ESP32-S3-DEVKITC-1-N8R2, symbol symbols:ESP32-S3-DEVKITC-SYMBOL
- J4: value PlugIn_Terminal_01x02 -> 5V_IN; footprint Library:steckklemme2x1_dnp -> Library:anschlussklemme2x1_3_5; symbol symbols:PlugIn_Terminal_01x02_dnp -> symbols:PlugIn_Terminal_Screw; MPN C8387 -> C695629
- renumbered C4 to C1, C19 to C10, C24 to C11, C27 to C12, C31 to C13, C33 to C14, C6 to C15, C14 to C16, C14 to C17, C17 to C18, C10 to C2, C21 to C3, C12 to C4, C6 to C5, C16 to C6, C14 to C7, C15 to C8, C17 to C9, Q4 to Q1, Q5 to Q2, R29 to R1, R37 to R10, R28 to R11, R36 to R12, R25 to R13, R34 to R15, R38 to R16, R39 to R17, R40 to R18, R41 to R19, R43 to R20, R45 to R21, R37 to R22, R25 to R23, R25 to R24, R36 to R25, R45 to R26, R22 to R28, R25 to R29, R30 to R3, R22 to R30, R25 to R31, R34 to R33, R31 to R4, R32 to R5, R34 to R6, R33 to R7, R25 to R8, R22 to R9, U4 to U1, U6 to U2, U5 to U3

Commit message: DIN board: 0402 passives, placement, planes, partial routing
Copied bus/audio sheet: 100 resistors and caps from 0603 to 0402 (JLC parts
updated); C1, C28-C31 (bus voltage) and C12 (10u on +5V) stay 0603.

Board: all 208 parts placed by block (bus top, W5500 behind RJ45, codec,
power/USB front), DNP options on the back. 4 layers: In1 GND, In2 +3.3V,
175 plane vias. Autorouted with KiCadRoutingTools; 34 connections still
open around the W5500 and the ES8374. DRC: 0 errors.

Co-Authored-By: Claude Opus 5.5 <noreply@anthropic.com>
Parts:
- C10: footprint Library:C_0603_1608Metric_Pad1.08x0.95mm_HandSolder -> Library:C_0402_1005Metric_Pad0.74x0.62mm_HandSolder; MPN C1588 -> C1523
- C14, C23, C25, C27, C35, C37, C39, C41, C43, C47, C52, C54, C56: footprint Library:C_0603_1608Metric_Pad1.08x0.95mm_HandSolder -> Library:C_0402_1005Metric_Pad0.74x0.62mm_HandSolder; MPN C96446 -> C15525
- C18, C2, C4, C8, C9: footprint Library:C_0603_1608Metric_Pad1.08x0.95mm_HandSolder -> Library:C_0402_1005Metric_Pad0.74x0.62mm_HandSolder; MPN C14858 -> C1546
- C22, C24, C26, C32, C33, C34: footprint Library:C_0603_1608Metric_Pad1.08x0.95mm_HandSolder -> Library:C_0402_1005Metric_Pad0.74x0.62mm_HandSolder; MPN C14663 -> C1525
- C44, C45, C48, C49, C50, C61: footprint Library:C_0603_1608Metric_Pad1.08x0.95mm_HandSolder -> Library:C_0402_1005Metric_Pad0.74x0.62mm_HandSolder; MPN C1653 -> C1555
- R1, R20: footprint Library:R_0603_1608Metric_Pad0.98x0.95mm_HandSolder -> Library:R_0402_1005Metric_Pad0.72x0.64mm_HandSolder; MPN C22795 -> C2909318
- R10, R15, R22, R27, R33, R6: footprint Library:R_0603_1608Metric_Pad0.98x0.95mm_HandSolder -> Library:R_0402_1005Metric_Pad0.72x0.64mm_HandSolder; MPN C25810 -> C2909327
- R11, R23, R24, R73: footprint Library:R_0603_1608Metric_Pad0.98x0.95mm_HandSolder -> Library:R_0402_1005Metric_Pad0.72x0.64mm_HandSolder; MPN C25804 -> C25744
- R12, R25, R46, R47: footprint Library:R_0603_1608Metric_Pad0.98x0.95mm_HandSolder -> Library:R_0402_1005Metric_Pad0.72x0.64mm_HandSolder; MPN C22940 -> C144772
- R14, R37, R38, R39, R40, R69, R70, R71, R72: footprint Library:R_0603_1608Metric_Pad0.98x0.95mm_HandSolder -> Library:R_0402_1005Metric_Pad0.72x0.64mm_HandSolder; MPN C21190 -> C11702
- R16, R17, R5, R7: footprint Library:R_0603_1608Metric_Pad0.98x0.95mm_HandSolder -> Library:R_0402_1005Metric_Pad0.72x0.64mm_HandSolder; MPN C23186 -> C25905
- R18, R19, R3, R35, R4: footprint Library:R_0603_1608Metric_Pad0.98x0.95mm_HandSolder -> Library:R_0402_1005Metric_Pad0.72x0.64mm_HandSolder; MPN C23254 -> C2909388
- R2: footprint Library:R_0603_1608Metric_Pad0.98x0.95mm_HandSolder -> Library:R_0402_1005Metric_Pad0.72x0.64mm_HandSolder; MPN C31850 -> C25768
- R21, R26: footprint Library:R_0603_1608Metric_Pad0.98x0.95mm_HandSolder -> Library:R_0402_1005Metric_Pad0.72x0.64mm_HandSolder; MPN C23162 -> C25900
- R28, R30, R9: footprint Library:R_0603_1608Metric_Pad0.98x0.95mm_HandSolder -> Library:R_0402_1005Metric_Pad0.72x0.64mm_HandSolder; MPN C25819 -> C25792
- R32: footprint Library:R_0603_1608Metric_Pad0.98x0.95mm_HandSolder -> Library:R_0402_1005Metric_Pad0.72x0.64mm_HandSolder; MPN C22962 -> C25092
- R34, R36, R55, R56, R57, R58, R59, R60, R61, R62, R63, R64, R65, R66, R67, R68, R74: footprint Library:R_0603_1608Metric_Pad0.98x0.95mm_HandSolder -> Library:R_0402_1005Metric_Pad0.72x0.64mm_HandSolder; MPN C21189 -> C17168
- R41, R42, R43, R44, R50, R51, R52, R53, R54: footprint Library:R_0603_1608Metric_Pad0.98x0.95mm_HandSolder -> Library:R_0402_1005Metric_Pad0.72x0.64mm_HandSolder; MPN C23140 -> C25105
- R48, R49: footprint Library:R_0603_1608Metric_Pad0.98x0.95mm_HandSolder -> Library:R_0402_1005Metric_Pad0.72x0.64mm_HandSolder; MPN C22775 -> C25076

Commit message: gdoor-din: finish routing, 0.45/0.2 mm vias, drop unused mic options
- Route every net: kicad-cli DRC reports 0 unconnected, 0 errors,
  schematic parity clean.
- Project rules: min via 0.45 mm / drill 0.2 mm (JLCPCB standard on
  4 layers), Default netclass track 0.2 mm, via 0.45/0.2.
- Schematic: remove the option parts C28, C30, R61-R66, R67/R68 and
  their dangling wiring; keep R69-R72 (attenuation) and C62/C63
  (filtering). No-connects on the unused U5 speaker pins.

Open: one 0.07 mm +3.3V dangling stub, silk clean-up, F/B GND pours.

Co-Authored-By: Claude Opus 5.5 <noreply@anthropic.com>
Parts:
- removed C28, C30: 10u, Library:C_0603_1608Metric_Pad1.08x0.95mm_HandSolder, symbol symbols:10u
- removed R61, R62, R63, R64, R65, R66, R67, R68: 0, Library:R_0402_1005Metric_Pad0.72x0.64mm_HandSolder, symbol symbols:0R
- renumbered C2 to C10, C4 to C12, C17 to C14, C16 to C14, C7 to C14, C8 to C15, C6 to C16, C18 to C17, C9 to C17, C10 to C19, C3 to C21, C11 to C24, C12 to C27, C13 to C31, C14 to C33, C1 to C4, C5 to C6, C15 to C6, Q1 to Q4, Q2 to Q5, R9 to R22, R28 to R22, R30 to R22, R8 to R25, R31 to R25, R29 to R25, R13 to R25, R23 to R25, R24 to R25, R11 to R28, R1 to R29, R3 to R30, R4 to R31, R5 to R32, R7 to R33, R6 to R34, R15 to R34, R33 to R34, R12 to R36, R25 to R36, R22 to R37, R10 to R37, R16 to R38, R17 to R39, R18 to R40, R19 to R41, R20 to R43, R26 to R45, R21 to R45, U1 to U4, U3 to U5, U2 to U6
Connections:
- no-connect marks 2 -> 4

Commit message: gdoor-din: 1210 part for the 100u caps, unify resistor values for JLC BOM
JLCPCB flagged two BOM problems:
- C19, C20, C59 sit on 1210 pads but carried C15008, a 1206 6.3 V part
  (CL31A107MQHNNNE; same mismatch upstream). Now C23742
  (CL32A107MPVNNNE, 100 uF 10 V X5R 1210), which also gives C20 on +5V
  a sensible voltage margin.
- One part matched several BOM lines because the copied sheet spelled
  values "5k1"/"4k7" and the new sheet "5.1k"/"4.7k". R5, R7, R16, R17
  are now 5.1k and R26 4.7k.

The copied sheet's symbols carry stale Reference properties from the
upstream sheet, so Konnect edited the wrong symbols; the edit was keyed
on each symbol's live instance instead and the file rewritten by
kicad-cli sch upgrade. Netlist diff: exactly these 8 fields.
DRC: 0 errors, 0 unconnected, parity clean.

Co-Authored-By: Claude Opus 5.5 <noreply@anthropic.com>
Parts:
- C19, C20, C59: MPN C15008 -> C23742
- R32, R33, R38, R39: value 5k1 -> 5.1k
- R45: value 4k7 -> 4.7k
Changed lines of the file:
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@@
 			)
 		)
-		(property "Value" "4k7"
+		(property "Value" "4.7k"
 			(at 133.35 61.595 90)
 			(show_name no)
@@
 			)
 		)
-		(property "Value" "5k1"
+		(property "Value" "5.1k"
 			(at 80.645 77.47 90)
 			(show_name no)
@@
 			)
 		)
-		(property "Value" "5k1"
+		(property "Value" "5.1k"
 			(at 118.11 157.48 90)
 			(show_name no)
@@
 			)
 		)
-		(property "Value" "5k1"
+		(property "Value" "5.1k"
 			(at 125.73 157.48 90)
 			(show_name no)
@@
 			)
 		)
-		(property "MPN" "C15008"
+		(property "MPN" "C23742"
 			(at 133.985 195.58 0)
 			(hide yes)
@@
 			)
 		)
-		(property "MPN" "C15008"
+		(property "MPN" "C23742"
 			(at 69.85 257.81 0)
 			(hide yes)
@@
 			)
 		)
-		(property "Value" "5k1"
+		(property "Value" "5.1k"
 			(at 74.295 77.47 90)
 			(show_name no)
@@
 			)
 		)
-		(property "MPN" "C15008"
+		(property "MPN" "C23742"
 			(at 146.05 215.9 0)
 			(hide yes)

Commit message: gdoor-din: logic check, drop unused options, flush USB-C cut-out
Logic check of the schematic against the netlist (ERC, block by block).
One real error: the BOOT/RESET labels were swapped. SW101 is EN (RESET),
SW102 is IO0 (BOOT). Fixed on the silkscreen and on the enclosure lid.

Removed the unfitted options that have no use on this board: R55
(+3.3V to +3.3V_AUDIO link), R56 (RX_DAC link), R69-R72 (mic
attenuation) and C62/C63 (alternative mic coupling), with their wiring
and their tracks (including a +3.3V_AUDIO run on In2.Cu that only served
R55). Netlist comparison: no remaining pin changed net. DRC: 0 errors,
0 unconnected. BOM and CPL unchanged (all were DNP).

Silkscreen labels RESET (SW101) and BOOT (SW102). Enclosure: the USB-C
opening is now a 9.4 x 3.7 mm stadium around the flush receptacle shell;
the fit check models the shell as a stadium too and is empty.

DESIGN.md rewritten: blocks, pin map, logic-check results, and open
points split into decisions (C10/R21/C18 DNP vs upstream, C29/C31 25 V
on the bus, 0 ohm links, J4/D2), KiCad to-dos (F8 for two renamed nets,
the RX_DAC bus entry) and first-build checks.

Co-Authored-By: Claude Opus 5.5 <noreply@anthropic.com>
Parts:
- removed C62, C63: 100n, Library:C_0402_1005Metric_Pad0.74x0.62mm_HandSolder, symbol symbols:100n_0402
- removed R55, R56: 0, Library:R_0402_1005Metric_Pad0.72x0.64mm_HandSolder, symbol symbols:0R
- removed R69, R70, R71, R72: 1k, Library:R_0402_1005Metric_Pad0.72x0.64mm_HandSolder, symbol symbols:1k

Commit message: gdoor-din: 50 V bus caps, fit C10/R21 on the front
C29 and C31 sit on the bus DC (up to about 30 V) through R74 and were
25 V parts. C29 is now 10 uF 50 V 1206 (C13585, like C21); C31 is
10 uF 50 V 0805 (C440198), since a 1206 does not fit at its spot. C31's
pad-1 route to R40 is re-routed down its right side.

C10 (1 nF) and R21 (4k7) on the TX node are fitted on the upstream
board but were DNP on B.Cu here. They are now on F.Cu, fitted by JLC,
joined to the old TX-node track by a via, with their own GND vias.
C18 (100 pF, TX driver input) has no free F.Cu spot and stays on B.Cu
for hand soldering.

Schematic: C10/R21 no longer DNP, the leftover RX_DAC bus entry is
removed; ERC has no errors. DRC: 0 errors, 0 unconnected, 0 parity.
JLC files regenerated: BOM 62 lines, CPL 186 parts.

Co-Authored-By: Claude Opus 5.5 <noreply@anthropic.com>
Parts:
- C10: renamed from C19; now fitted
- C29: footprint Library:C_0603_1608Metric_Pad1.08x0.95mm_HandSolder -> Capacitor_SMD:C_1206_3216Metric; MPN C96446 -> C13585
- C31: footprint Library:C_0603_1608Metric_Pad1.08x0.95mm_HandSolder -> Capacitor_SMD:C_0805_2012Metric; MPN C96446 -> C440198
- R21: renamed from R45; now fitted
- renumbered C4 to C1, C24 to C11, C27 to C12, C31 to C13, C33 to C14, C6 to C15, C14 to C16, C14 to C17, C17 to C18, C10 to C2, C21 to C3, C12 to C4, C6 to C5, C16 to C6, C14 to C7, C15 to C8, C17 to C9, Q4 to Q1, Q5 to Q2, R29 to R1, R37 to R10, R28 to R11, R36 to R12, R25 to R13, R34 to R15, R38 to R16, R39 to R17, R40 to R18, R41 to R19, R43 to R20, R37 to R22, R25 to R23, R25 to R24, R36 to R25, R45 to R26, R22 to R28, R25 to R29, R30 to R3, R22 to R30, R25 to R31, R34 to R33, R31 to R4, R32 to R5, R34 to R6, R33 to R7, R25 to R8, R22 to R9, U4 to U1, U6 to U2, U5 to U3
