File: hardware/boards/din/esp32.kicad_pcb (KiCad board)
At the start: 4 copper layers, 56.8 x 85 mm, 190 parts, among them J1 PlugIn_Terminal_Screw, J101 USB-C, J102 HR911105A, J103 EXP, J4 5V_IN, Q1 MMBT5401, Q2 MMBT2222A, SW101 TL3342, SW102 TL3342, U1 TLV9351, U101 ESP32-S3-WROOM-1-N8R2, U102 USBLC6-2SC6, U103 AP2114H-3.3TRG1, U104 W5500, U2 LMV321, U3 LMV321, U5 ES8374, U6 LM393, U7 AMS1117-3.3, Y101 25MHz

Commit message: gdoor-din: cut JLC Extended-part fees from $60 to $21
Hand-soldered and left off the JLC order (jlcfab.py HAND_SOLDERED): J1,
J102, U103, U102, U2/U3, C19/C20/C59, Y101.

No-fee parts instead of Extended ones (schematic, board fields, DESIGN.md):
- 18k, 2.4k, 6.8 nF: same values as Preferred parts C25762/C25882/C1542
- 82k -> 100k Basic C25741: R3/R4 and R18/R19 are 1:1 reference dividers;
  R35 makes the bus-voltage divider 100k/10k (/11, about 34 V full scale)
- R112/R113/R117/R118 3.3 ohm -> 0 ohm: series resistors between the W5500
  and its 49.9 ohm terminations
- D103 green -> red C2286, R105 100 ohm -> 1k so both LEDs run ~1.3 mA

Still Extended: U1, U5, U101, U104, J101, R1/R20 (130k), R108 (12.4k).
Also a root .gitignore for .vscode/.

Co-Authored-By: Claude Opus 5.5 <noreply@anthropic.com>
Parts:
- D103: value green -> red
- R105: value 100 -> 1k
- R112, R113, R117, R118: value 3.3 -> 0
- R18, R19, R3, R35, R4: value 82k -> 100k
Changed lines of the file:
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@@
 			)
 		)
-		(property "Value" "100"
+		(property "Value" "1k"
 			(at 0 1.17 90)
 			(layer "F.Fab")
@@
 			)
 		)
-		(property "LCSC" "C25076"
+		(property "LCSC" "C11702"
 			(at 0 0 90)
 			(unlocked yes)
@@
 			)
 		)
-		(property "Value" "3.3"
+		(property "Value" "0"
 			(at 0 1.17 270)
 			(layer "F.Fab")
@@
 			)
 		)
-		(property "LCSC" "C2933094"
+		(property "LCSC" "C17168"
 			(at 0 0 270)
 			(unlocked yes)
@@
 			)
 		)
-		(property "Value" "82k"
+		(property "Value" "100k"
 			(at 0 1.17 90)
 			(layer "F.Fab")
@@
 			)
 		)
-		(property "MPN" "C2909388"
+		(property "MPN" "C25741"
 			(at 0 0 90)
 			(layer "F.SilkS")
@@
 			)
 		)
-		(property "MPN" "C2909327"
+		(property "MPN" "C25762"
 			(at 0 0 0)
 			(layer "F.SilkS")
@@
 			)
 		)
-		(property "MPN" "C144772"
+		(property "MPN" "C25882"
 			(at 0 0 0)
 			(layer "F.SilkS")
@@
 			)
 		)
-		(property "MPN" "C2909327"
+		(property "MPN" "C25762"
 			(at 0 0 0)
 			(layer "F.SilkS")
@@
 			)
 		)
-		(property "Value" "82k"
+		(property "Value" "100k"
 			(at 0 1.17 90)
 			(layer "F.Fab")
@@
 			)
 		)
-		(property "MPN" "C2909388"
+		(property "MPN" "C25741"
 			(at 0 0 90)
 			(layer "F.SilkS")
@@
 			)
 		)
-		(property "MPN" "C144772"
+		(property "MPN" "C25882"
 			(at 0 0 0)
 			(layer "F.SilkS")
@@
 			)
 		)
-		(property "Value" "3.3"
+		(property "Value" "0"
 			(at 0 1.17 0)
 			(layer "F.Fab")
@@
 			)
 		)
-		(property "LCSC" "C2933094"
+		(property "LCSC" "C17168"
 			(at 0 0 0)
 			(unlocked yes)
@@
 			)
 		)
-		(property "LCSC" "C93654"
+		(property "LCSC" "C1542"
 			(at 0 0 0)
 			(unlocked yes)
@@
 			)
 		)
-		(property "Value" "3.3"
+		(property "Value" "0"
 			(at 0 1.17 270)
 			(layer "F.Fab")
@@
 			)
 		)
-		(property "LCSC" "C2933094"
+		(property "LCSC" "C17168"
 			(at 0 0 270)
 			(unlocked yes)
@@
 			)
 		)
-		(property "Value" "82k"
+		(property "Value" "100k"
 			(at 0 1.17 0)
 			(layer "F.Fab")
@@
 			)
 		)
-		(property "MPN" "C2909388"
+		(property "MPN" "C25741"
 			(at 0 0 0)
 			(layer "F.SilkS")
@@
 			)
 		)
-		(property "MPN" "C2909327"
+		(property "MPN" "C25762"
 			(at 0 0 0)
 			(layer "F.SilkS")
@@
 			)
 		)
-		(property "MPN" "C2909327"
+		(property "MPN" "C25762"
 			(at 0 0 90)
 			(layer "F.SilkS")
@@
 			)
 		)
-		(property "Value" "82k"
+		(property "Value" "100k"
 			(at 0 1.17 90)
 			(layer "F.Fab")
@@
 			)
 		)
-		(property "MPN" "C2909388"
+		(property "MPN" "C25741"
 			(at 0 0 90)
 			(layer "F.SilkS")
@@
 			)
 		)
-		(property "MPN" "C2909327"
+		(property "MPN" "C25762"
 			(at 0 0 0)
 			(layer "F.SilkS")
@@
 			)
 		)
-		(property "Value" "3.3"
+		(property "Value" "0"
 			(at 0 1.17 0)
 			(layer "F.Fab")
@@
 			)
 		)
-		(property "LCSC" "C2933094"
+		(property "LCSC" "C17168"
 			(at 0 0 0)
 			(unlocked yes)
@@
 			)
 		)
-		(property "Value" "green"
+		(property "Value" "red"
 			(at 0 1.43 0)
 			(layer "F.Fab")
@@
 			)
 		)
-		(property "LCSC" "C12624"
+		(property "LCSC" "C2286"
 			(at 0 0 0)
 			(unlocked yes)
@@
 			)
 		)
-		(property "Value" "82k"
+		(property "Value" "100k"
 			(at 0 1.17 90)
 			(layer "F.Fab")
@@
 			)
 		)
-		(property "MPN" "C2909388"
+		(property "MPN" "C25741"
 			(at 0 0 90)
 			(layer "F.SilkS")
@@
 			)
 		)
-		(property "LCSC" "C93654"
+		(property "LCSC" "C1542"
 			(at 0 0 0)
 			(unlocked yes)
@@
 			)
 		)
-		(property "MPN" "C144772"
+		(property "MPN" "C25882"
 			(at 0 0 90)
 			(layer "F.SilkS")
@@
 			)
 		)
-		(property "MPN" "C144772"
+		(property "MPN" "C25882"
 			(at 0 0 0)
 			(layer "F.SilkS")
@@
 			)
 		)
-		(property "MPN" "C2909327"
+		(property "MPN" "C25762"
 			(at 0 0 90)
 			(layer "F.SilkS")

Commit message: gdoor-din: R3/R4 back to 82k, RX band-pass oscillated with 100k
R3/R4 are the ground leg of the RX Sallen-Key band-pass (U2, gain 1.94),
not only a 1.65 V divider. With 100k (7ce317d) its damping goes negative
and the stage oscillates at ~49 kHz with no bus signal; it is stable
below ~90k. Back to 82k (C2909388, Extended, as upstream esp32-mini).
JLC has no fee-free 82k in 0402. R18/R19 stay 100k: the TX stage
(gain 1.39) is stable and its peak moves onto the 52 kHz carrier.

Add spice/: ngspice testbench of the bus side on KiCad's ngspice.dll
(RX/TX filters, comparator, +5V_onoff switch, codec coupling, hot-plug),
results and plots in spice/README.md. Production files regenerated
(BOM change only; gerbers differ in timestamps).

Co-Authored-By: Claude Opus 5.5 <noreply@anthropic.com>
Parts:
- R3, R4: value 100k -> 82k
Changed lines of the file:
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@@
 			)
 		)
-		(property "Value" "100k"
+		(property "Value" "82k"
 			(at 0 1.17 90)
 			(layer "F.Fab")
@@
 			)
 		)
-		(property "MPN" "C25741"
+		(property "MPN" "C2909388"
 			(at 0 0 90)
 			(layer "F.SilkS")
@@
 			)
 		)
-		(property "Value" "100k"
+		(property "Value" "82k"
 			(at 0 1.17 90)
 			(layer "F.Fab")
@@
 			)
 		)
-		(property "MPN" "C25741"
+		(property "MPN" "C2909388"
 			(at 0 0 90)
 			(layer "F.SilkS")

Commit message: gdoor-din: crystal caps 18 pF -> 33 pF, Ethernet front-end simulation
Y101 (C164045) is rated for CL = 20 pF; C108/C109 at 18 pF gave only
12-14 pF with stray, pulling the 25 MHz clock +35..+55 ppm (802.3u
allows +-50 ppm). 33 pF (C1562, JLC Basic) keeps it within +-7 ppm.

Add spice/eth_sim.py: W5500 + HR911105A front end (magjack fitted to
typical 10/100 figures). Return loss passes 802.3 on both pairs (~3.5 dB
margin), ~40 mA TX current gives the nominal 1.0 V MLT-3 level, FB101
has no resonance problem, C121/C122 put the RX low corner at 220 kHz as
in WIZnet's reference. plot.py's svg_plot is now importable.

Production files regenerated (BOM change only; gerbers differ in
timestamps).

Co-Authored-By: Claude Opus 5.5 <noreply@anthropic.com>
Parts:
- C108, C109: value 18p -> 33p
Changed lines of the file:
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@@
 			)
 		)
-		(property "Value" "18p"
+		(property "Value" "33p"
 			(at 0 1.16 180)
 			(layer "F.Fab")
@@
 			)
 		)
-		(property "LCSC" "C1549"
+		(property "LCSC" "C1562"
 			(at 0 0 180)
 			(unlocked yes)
@@
 			)
 		)
-		(property "Value" "18p"
+		(property "Value" "33p"
 			(at 0 1.16 90)
 			(layer "F.Fab")
@@
 			)
 		)
-		(property "LCSC" "C1549"
+		(property "LCSC" "C1562"
 			(at 0 0 90)
 			(unlocked yes)
