File: hardware/boards/din/esp32.kicad_pcb (KiCad board)
At the start: 4 copper layers, 56.8 x 85 mm, 191 parts, among them J1 PlugIn_Terminal_Screw, J101 USB-C, J102 HR911105A, J103 EXP, J4 5V_IN, Q1 MMBT5401, Q2 MMBT2222A, SW101 TL3342, SW102 TL3342, U1 TLV9351, U101 ESP32-S3-WROOM-1-N8R2, U102 USBLC6-2SC6, U103 AP2114H-3.3TRG1, U104 W5500, U2 LMV321, U3 LMV321, U5 ES8374, U6 LM393, U7 AMS1117-3.3, Y101 25MHz

Commit message: gdoor-din: J102 to HanRun HY911105AE (C69427)
HR911105A (C12074) is out of stock at LCSC. HY911105AE is HanRun's
-40..+85 C version of the same jack: same pinout, LEDs, magnetics and
hole pattern, so the footprint stays. Updates the LCSC field, value and
datasheet, and the BOM, hand-solder and price files.

Co-Authored-By: Claude Opus 5.5 <noreply@anthropic.com>
Parts:
- J102: value HR911105A -> HY911105AE
Changed lines of the file:
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@@
 			)
 		)
-		(property "Value" "HR911105A"
+		(property "Value" "HY911105AE"
 			(at 4.44 18.5 270)
 			(layer "F.Fab")
@@
 			)
 		)
-		(property "Datasheet" ""
+		(property "Datasheet" "https://www.lcsc.com/datasheet/C69427.pdf"
 			(at 0 0 270)
 			(unlocked yes)
@@
 			)
 		)
-		(property "LCSC" "C12074"
+		(property "LCSC" "C69427"
 			(at 0 0 270)
 			(unlocked yes)
