File: hardware/boards/din/esp32.kicad_sch (KiCad schematic)
At the start: 130 parts, among them J1 PlugIn_Terminal_Screw, J4 5V_IN, Q1 MMBT5401, Q2 MMBT2222A, U1 TLV9351, U2 LMV321, U3 LMV321, U5 ES8374, U6 LM393, U7 AMS1117-3.3

Commit message: gdoor-din: cut JLC Extended-part fees from $60 to $21
Hand-soldered and left off the JLC order (jlcfab.py HAND_SOLDERED): J1,
J102, U103, U102, U2/U3, C19/C20/C59, Y101.

No-fee parts instead of Extended ones (schematic, board fields, DESIGN.md):
- 18k, 2.4k, 6.8 nF: same values as Preferred parts C25762/C25882/C1542
- 82k -> 100k Basic C25741: R3/R4 and R18/R19 are 1:1 reference dividers;
  R35 makes the bus-voltage divider 100k/10k (/11, about 34 V full scale)
- R112/R113/R117/R118 3.3 ohm -> 0 ohm: series resistors between the W5500
  and its 49.9 ohm terminations
- D103 green -> red C2286, R105 100 ohm -> 1k so both LEDs run ~1.3 mA

Still Extended: U1, U5, U101, U104, J101, R1/R20 (130k), R108 (12.4k).
Also a root .gitignore for .vscode/.

Co-Authored-By: Claude Opus 5.5 <noreply@anthropic.com>
Parts:
- R10, R15, R22, R27, R33, R6: MPN C2909327 -> C25762
- R12, R25, R46, R47: MPN C144772 -> C25882
- R18, R19, R3, R35, R4: value 82k -> 100k; MPN C2909388 -> C25741
Changed lines of the file:
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@@
 			)
 		)
-		(property "MPN" "C2909327"
+		(property "MPN" "C25762"
 			(at 130.81 104.14 0)
 			(hide yes)
@@
 			)
 		)
-		(property "Value" "82k"
+		(property "Value" "100k"
 			(at 127 137.16 90)
 			(show_name no)
@@
 			)
 		)
-		(property "MPN" "C2909388"
+		(property "MPN" "C25741"
 			(at 127 137.16 0)
 			(hide yes)
@@
 			)
 		)
-		(property "MPN" "C2909327"
+		(property "MPN" "C25762"
 			(at 74.93 158.75 0)
 			(hide yes)
@@
 			)
 		)
-		(property "MPN" "C2909327"
+		(property "MPN" "C25762"
 			(at 109.22 120.015 0)
 			(hide yes)
@@
 			)
 		)
-		(property "MPN" "C144772"
+		(property "MPN" "C25882"
 			(at 92.075 69.85 0)
 			(hide yes)
@@
 			)
 		)
-		(property "Value" "82k"
+		(property "Value" "100k"
 			(at 127 129.54 90)
 			(show_name no)
@@
 			)
 		)
-		(property "MPN" "C2909388"
+		(property "MPN" "C25741"
 			(at 127 129.54 0)
 			(hide yes)
@@
 			)
 		)
-		(property "MPN" "C144772"
+		(property "MPN" "C25882"
 			(at 203.2 113.03 0)
 			(hide yes)
@@
 			)
 		)
-		(property "MPN" "C144772"
+		(property "MPN" "C25882"
 			(at 197.485 113.03 0)
 			(hide yes)
@@
 			)
 		)
-		(property "Value" "82k"
+		(property "Value" "100k"
 			(at 203.2 48.26 90)
 			(show_name no)
@@
 			)
 		)
-		(property "MPN" "C2909388"
+		(property "MPN" "C25741"
 			(at 203.2 48.26 0)
 			(hide yes)
@@
 			)
 		)
-		(property "MPN" "C2909327"
+		(property "MPN" "C25762"
 			(at 130.81 99.06 0)
 			(hide yes)
@@
 			)
 		)
-		(property "Value" "82k"
+		(property "Value" "100k"
 			(at 71.755 54.61 90)
 			(show_name no)
@@
 			)
 		)
-		(property "MPN" "C2909388"
+		(property "MPN" "C25741"
 			(at 71.755 54.61 0)
 			(hide yes)
@@
 			)
 		)
-		(property "Value" "82k"
+		(property "Value" "100k"
 			(at 71.755 46.99 90)
 			(show_name no)
@@
 			)
 		)
-		(property "MPN" "C2909388"
+		(property "MPN" "C25741"
 			(at 71.755 46.99 0)
 			(hide yes)
@@
 			)
 		)
-		(property "MPN" "C2909327"
+		(property "MPN" "C25762"
 			(at 80.01 158.75 0)
 			(hide yes)
@@
 			)
 		)
-		(property "MPN" "C144772"
+		(property "MPN" "C25882"
 			(at 120.65 62.23 0)
 			(hide yes)
@@
 			)
 		)
-		(property "MPN" "C2909327"
+		(property "MPN" "C25762"
 			(at 90.805 35.56 0)
 			(hide yes)

Commit message: gdoor-din: R3/R4 back to 82k, RX band-pass oscillated with 100k
R3/R4 are the ground leg of the RX Sallen-Key band-pass (U2, gain 1.94),
not only a 1.65 V divider. With 100k (7ce317d) its damping goes negative
and the stage oscillates at ~49 kHz with no bus signal; it is stable
below ~90k. Back to 82k (C2909388, Extended, as upstream esp32-mini).
JLC has no fee-free 82k in 0402. R18/R19 stay 100k: the TX stage
(gain 1.39) is stable and its peak moves onto the 52 kHz carrier.

Add spice/: ngspice testbench of the bus side on KiCad's ngspice.dll
(RX/TX filters, comparator, +5V_onoff switch, codec coupling, hot-plug),
results and plots in spice/README.md. Production files regenerated
(BOM change only; gerbers differ in timestamps).

Co-Authored-By: Claude Opus 5.5 <noreply@anthropic.com>
Parts:
- R3, R4: value 100k -> 82k; MPN C25741 -> C2909388
Changed lines of the file:
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@@
 			)
 		)
-		(property "Value" "100k"
+		(property "Value" "82k"
 			(at 71.755 54.61 90)
 			(show_name no)
@@
 			)
 		)
-		(property "MPN" "C25741"
+		(property "MPN" "C2909388"
 			(at 71.755 54.61 0)
 			(hide yes)
@@
 			)
 		)
-		(property "Value" "100k"
+		(property "Value" "82k"
 			(at 71.755 46.99 90)
 			(show_name no)
@@
 			)
 		)
-		(property "MPN" "C25741"
+		(property "MPN" "C2909388"
 			(at 71.755 46.99 0)
 			(hide yes)

Commit message: gdoor-din: four JLC Extended parts made fee-free, values kept
Saves $12 of JLC's $3-per-type Extended loading fee (8 charged types -> 4).

- R3/R4 82k: 0402 C2909388 -> 0603 C23254 (Basic).
- R1/R20 130k: 0402 C2909318 -> 0603 C22795 (Preferred Extended).
  The larger pads needed two small reroutes: Net-(J1-Pin_2) between R3
  and R5, and the Net-(C8-Pad2) diagonal next to R20.
- R108 12.4k 1% (C2929935) -> R108 10k (C25744) + new R123 2.4k
  (C25882) in series, node ETH_EXRES_LO; 12.4k exactly. R123 sits below
  R108; the GND via beside R108 pad 2 moved to R123 pad 2.
- Y101 C164045 (CL 20 pF, +-50 ppm) -> C9006 (CL 12 pF, +-20 ppm, Basic),
  same 3225 footprint; C108/C109 33 pF -> 15 pF (C1548). eth_sim.py puts
  the pull at -5.5..+18.5 ppm, worst case ~+48.5 ppm with tolerance and
  temperature, inside 802.3u's +-50 ppm.

DRC (zone refill): 0 errors, 0 unconnected, schematic parity clean.
Production files regenerated with jlcfab.py. mcu_eth.kicad_sch was
rewritten in compact s-expression layout by the Konnect schematic tool;
a netlist comparison shows only the changes above.

Also contains an unrelated one-line change from another session: J101's
3D-model offset (y 0.294 -> -1.045) in esp32.kicad_pcb.

Co-Authored-By: Claude Opus 5.5 <noreply@anthropic.com>
Parts:
- R1, R20: footprint Library:R_0402_1005Metric_Pad0.72x0.64mm_HandSolder -> Resistor_SMD:R_0603_1608Metric; MPN C2909318 -> C22795
- R3, R4: footprint Library:R_0402_1005Metric_Pad0.72x0.64mm_HandSolder -> Resistor_SMD:R_0603_1608Metric; MPN C2909388 -> C23254
Changed lines of the file:
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@@
 			)
 		)
-		(property "Footprint" "Library:R_0402_1005Metric_Pad0.72x0.64mm_HandSolder"
+		(property "Footprint" "Resistor_SMD:R_0603_1608Metric"
 			(at 73.533 54.61 90)
 			(hide yes)
@@
 			)
 		)
-		(property "MPN" "C2909388"
+		(property "MPN" "C23254"
 			(at 71.755 54.61 0)
 			(hide yes)
@@
 			)
 		)
-		(property "Footprint" "Library:R_0402_1005Metric_Pad0.72x0.64mm_HandSolder"
+		(property "Footprint" "Resistor_SMD:R_0603_1608Metric"
 			(at 73.533 46.99 90)
 			(hide yes)
@@
 			)
 		)
-		(property "MPN" "C2909388"
+		(property "MPN" "C23254"
 			(at 71.755 46.99 0)
 			(hide yes)
@@
 			)
 		)
-		(property "Footprint" "Library:R_0402_1005Metric_Pad0.72x0.64mm_HandSolder"
+		(property "Footprint" "Resistor_SMD:R_0603_1608Metric"
 			(at 51.435 57.658 90)
 			(hide yes)
@@
 			)
 		)
-		(property "MPN" "C2909318"
+		(property "MPN" "C22795"
 			(at 51.435 55.88 0)
 			(hide yes)
@@
 			)
 		)
-		(property "Footprint" "Library:R_0402_1005Metric_Pad0.72x0.64mm_HandSolder"
+		(property "Footprint" "Resistor_SMD:R_0603_1608Metric"
 			(at 146.05 140.208 90)
 			(hide yes)
@@
 			)
 		)
-		(property "MPN" "C2909318"
+		(property "MPN" "C22795"
 			(at 146.05 138.43 0)
 			(hide yes)

Commit message: gdoor-din: every part gets a 0.5 mm designator, J4 fitted
Designators shrink from 0.8/0.12 to 0.5/0.1 mm and all 190 are shown,
each placed next to its part clear of pads, other silkscreen and the
other parts' bodies. The DRU and project text-height minimums follow.
The MPN fields that printed on R1, R3, R4 and R20 are hidden.

The screw terminals get labels: J4 "-", "+" and "5V" under its pins,
J1 "~" on both sides and "BUS" (the MB10S bridge makes it polarity-free).

J4 is no longer DNP or excluded from the BOM, in schematic and board.
It joins J1 in jlcfab.py's HAND_SOLDERED, so the JLC BOM and CPL are
unchanged.

Co-Authored-By: Claude Opus 5.5 <noreply@anthropic.com>
Parts:
- J4: now fitted; now in the parts list
Changed lines of the file:
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@@
 		(body_style 1)
 		(exclude_from_sim no)
-		(in_bom no)
+		(in_bom yes)
 		(on_board yes)
 		(in_pos_files yes)
-		(dnp yes)
+		(dnp no)
 		(fields_autoplaced yes)
 		(property "Reference" "J4"
